Commit message: Arm naming standarization

File: tiago_dual_description/robots/tiago_dual.urdf.xacro (robot description, xacro)
@@ -15,7 +15,7 @@
   <!-- ARGUMENTS -->
   <!-- tiago-arm, no-arm -->
-  <xacro:arg name="arm_left" default="tiago-arm"/>
+  <xacro:arg name="arm_model_left" default="tiago-arm"/>
   <!-- tiago-arm, no-arm -->
-  <xacro:arg name="arm_right" default="tiago-arm"/>
+  <xacro:arg name="arm_model_right" default="tiago-arm"/>
   <xacro:arg name="wrist_model_left" default="wrist-2010"/>
   <xacro:arg name="wrist_model_right" default="wrist-2010"/>
@@ -42,6 +42,6 @@
   <xacro:arg name="multiple" default="false"/>
   <!-- PROPERTIES -->
-  <xacro:property name="arm_left" value="$(arg arm_left)"/>
-  <xacro:property name="arm_right" value="$(arg arm_right)"/>
+  <xacro:property name="arm_model_left" value="$(arg arm_model_left)"/>
+  <xacro:property name="arm_model_right" value="$(arg arm_model_right)"/>
   <xacro:property name="wrist_model_left" value="$(arg wrist_model_left)" />
   <xacro:property name="wrist_model_right" value="$(arg wrist_model_right)" />
@@ -59,10 +59,10 @@
   <xacro:property name="head_link_name" value="head_2_link"/>
   <xacro:property name="description_calibration_dir" value="${arg description_calibration_dir}"/>
-  <xacro:property name="has_arm_left" value="${arm_left != 'no-arm'}"/>
+  <xacro:property name="has_arm_left" value="${arm_model_left != 'no-arm'}"/>
   <xacro:property name="has_ft_sensor_left" value="${ft_sensor_left != 'no-ft-sensor'}"/>
   <xacro:property name="has_end_effector_left" value="${end_effector_left not in ['false', 'False', 'no-ee']}"/>
   <xacro:property name="end_effector_left_link" value="${'wrist_left_ft_tool_link' if has_ft_sensor_left else 'arm_left_tool_link'}"/>
   <xacro:property name="end_effector_left_name" value="${'hand_left' if end_effector_left == 'pal-hey5' else 'gripper_left'}"/>
-  <xacro:property name="has_arm_right" value="${arm_right != 'no-arm'}"/>
+  <xacro:property name="has_arm_right" value="${arm_model_right != 'no-arm'}"/>
   <xacro:property name="has_ft_sensor_right" value="${ft_sensor_right != 'no-ft-sensor'}"/>
   <xacro:property name="has_end_effector_right" value="${end_effector_right not in ['false', 'False', 'no-ee']}"/>
@@ -70,9 +70,9 @@
   <xacro:property name="end_effector_right_name" value="${'hand_right' if end_effector_right == 'pal-hey5' else 'gripper_right'}"/>
   <!-- Properties check -->
-  <xacro:if value="${arm_left not in ['no-arm', 'tiago-arm']}">
-    <xacro:wrong_arm_left_type/>
+  <xacro:if value="${arm_model_left not in ['no-arm', 'tiago-arm']}">
+    <xacro:wrong_arm_model_left/>
   </xacro:if>
-  <xacro:if value="${arm_right not in ['no-arm', 'tiago-arm']}">
-    <xacro:wrong_arm_right_type/>
+  <xacro:if value="${arm_model_right not in ['no-arm', 'tiago-arm']}">
+    <xacro:wrong_arm_model_right/>
   </xacro:if>
   <xacro:if value="${wrist_model_left not in ['wrist-2010', 'wrist-2017']}">

File: tiago_dual_description/ros2_control/ros2_control.urdf.xacro (robot description, xacro)
@@ -12,9 +12,8 @@
   limitations under the License.
  -->
-<robot xmlns:xacro="http://ros.org/wiki/xacro"
-       name="tiago_dual" >
+<robot xmlns:xacro="http://ros.org/wiki/xacro" name="tiago_dual">
   <xacro:macro name="tiago_dual_ros2_control" params="use_sim:=^|false">
-    <xacro:arg name="arm_left" default="tiago-arm"/>
-    <xacro:arg name="arm_right" default="tiago-arm"/>
+    <xacro:arg name="arm_model_left" default="tiago-arm"/>
+    <xacro:arg name="arm_model_right" default="tiago-arm"/>
     <xacro:arg name="end_effector_left" default="pal-gripper"/>
     <xacro:arg name="end_effector_right" default="pal-gripper"/>
@@ -22,6 +21,6 @@
     <xacro:arg name="ft_sensor_right" default="no-ft-sensor"/>
     <xacro:arg name="description_calibration_dir" default="$(find tiago_dual_description)/urdf/calibration" />
-    <xacro:property name="has_arm_left" value="${arm_left != 'no-arm'}" />
-    <xacro:property name="has_arm_right" value="${arm_right != 'no-arm'}" />
+    <xacro:property name="has_arm_left" value="${arm_model_left != 'no-arm'}" />
+    <xacro:property name="has_arm_right" value="${arm_model_right != 'no-arm'}" />
     <xacro:property name="end_effector_left" value="$(arg end_effector_left)" />
     <xacro:property name="end_effector_right" value="$(arg end_effector_right)" />
@@ -76,8 +75,5 @@
         <!-- wrist -->
         <xacro:ros2_control_wrist_rotational name="arm_left_5" reduction="1.0" offset="${arm_left_5_joint_offset}" />
-        <xacro:ros2_control_wrist_differential name="arm_left" number_1="6" number_2="7"
-                                               act_reduction_1="-1.0" act_reduction_2="1.0"
-                                               jnt_reduction_1="1.0" jnt_reduction_2="1.0"
-                                               number_1_offset="${arm_left_6_joint_offset}" number_2_offset="${arm_left_7_joint_offset}" />
+        <xacro:ros2_control_wrist_differential name="arm_left" number_1="6" number_2="7" act_reduction_1="-1.0" act_reduction_2="1.0" jnt_reduction_1="1.0" jnt_reduction_2="1.0" number_1_offset="${arm_left_6_joint_offset}" number_2_offset="${arm_left_7_joint_offset}" />
         <xacro:if value="${end_effector_left == 'pal-gripper'}">
           <!-- pal-gripper -->
@@ -106,8 +102,5 @@
         <!-- wrist -->
         <xacro:ros2_control_wrist_rotational name="arm_right_5" reduction="1.0" offset="${arm_right_5_joint_offset}" />
-        <xacro:ros2_control_wrist_differential name="arm_right" number_1="6" number_2="7"
-                                               act_reduction_1="-1.0" act_reduction_2="1.0"
-                                               jnt_reduction_1="1.0" jnt_reduction_2="-1.0"
-                                               number_1_offset="${arm_right_6_joint_offset}" number_2_offset="${arm_right_7_joint_offset}" />
+        <xacro:ros2_control_wrist_differential name="arm_right" number_1="6" number_2="7" act_reduction_1="-1.0" act_reduction_2="1.0" jnt_reduction_1="1.0" jnt_reduction_2="-1.0" number_1_offset="${arm_right_6_joint_offset}" number_2_offset="${arm_right_7_joint_offset}" />
         <xacro:if value="${end_effector_right == 'pal-gripper'}">
           <!-- pal-gripper -->

Commit message: Changed arm_model to arm_type in the URDF

File: tiago_dual_description/robots/tiago_dual.urdf.xacro (robot description, xacro)
@@ -30,7 +30,7 @@
   <xacro:arg name="has_screen" default="false"/>
   <!-- no-arm, tiago-arm -->
-  <xacro:arg name="arm_model_left" default="tiago-arm"/>
+  <xacro:arg name="arm_type_left" default="tiago-arm"/>
   <!-- no-arm, tiago-arm -->
-  <xacro:arg name="arm_model_right" default="tiago-arm"/>
+  <xacro:arg name="arm_type_right" default="tiago-arm"/>
   <!--no-ft-sensor, schunk-ft -->
   <xacro:arg name="ft_sensor_left" default="schunk-ft"/>
@@ -62,6 +62,6 @@
   <xacro:property name="base_type" value="$(arg base_type)" />
   <xacro:property name="laser_model" value="$(arg laser_model)" />
-  <xacro:property name="arm_model_left" value="$(arg arm_model_left)"/>
-  <xacro:property name="arm_model_right" value="$(arg arm_model_right)"/>
+  <xacro:property name="arm_type_left" value="$(arg arm_type_left)"/>
+  <xacro:property name="arm_type_right" value="$(arg arm_type_right)"/>
   <xacro:property name="ft_sensor_left" value="$(arg ft_sensor_left)" />
   <xacro:property name="ft_sensor_right" value="$(arg ft_sensor_right)" />
@@ -81,9 +81,9 @@
     <xacro:wrong_laser_model/>
   </xacro:if>
-  <xacro:if value="${arm_model_left not in ['no-arm', 'tiago-arm']}">
-    <xacro:wrong_arm_model_left/>
-  </xacro:if>
-  <xacro:if value="${arm_model_right not in ['no-arm', 'tiago-arm']}">
-    <xacro:wrong_arm_model_right/>
+  <xacro:if value="${arm_type_left not in ['no-arm', 'tiago-arm']}">
+    <xacro:wrong_arm_type_left/>
+  </xacro:if>
+  <xacro:if value="${arm_type_right not in ['no-arm', 'tiago-arm']}">
+    <xacro:wrong_arm_type_right/>
   </xacro:if>
   <xacro:if value="${wrist_model_left not in ['wrist-2010', 'wrist-2017']}">
@@ -109,10 +109,10 @@
   </xacro:if>
   <!-- HW configuration helpers-->
-  <xacro:property name="has_arm_left" value="${arm_model_left != 'no-arm'}"/>
+  <xacro:property name="has_arm_left" value="${arm_type_left != 'no-arm'}"/>
   <xacro:property name="has_ft_sensor_left" value="${ft_sensor_left != 'no-ft-sensor'}"/>
   <xacro:property name="has_end_effector_left" value="${end_effector_left != 'no-end-effector'}"/>
   <xacro:property name="end_effector_left_link" value="${'wrist_left_ft_tool_link' if has_ft_sensor_left else 'arm_left_tool_link'}"/>
   <xacro:property name="end_effector_left_name" value="${'hand_left' if end_effector_left == 'pal-hey5' else 'gripper_left'}"/>
-  <xacro:property name="has_arm_right" value="${arm_model_right != 'no-arm'}"/>
+  <xacro:property name="has_arm_right" value="${arm_type_right != 'no-arm'}"/>
   <xacro:property name="has_ft_sensor_right" value="${ft_sensor_right != 'no-ft-sensor'}"/>
   <xacro:property name="has_end_effector_right" value="${end_effector_right != 'no-end-effector'}"/>

Commit message: add missing argument is_public_sim

File: tiago_dual_description/robots/tiago_dual.urdf.xacro (robot description, xacro)
@@ -58,4 +58,5 @@
   <xacro:arg name="is_multiple" default="false"/>
   <xacro:arg name="namespace" default=""/>
+  <xacro:arg name="is_public_sim" default="false"/>
   <!-- PROPERTIES -->
   <!-- HW configuration -->
@@ -126,4 +127,5 @@
   <xacro:property name="is_multiple" value="$(arg is_multiple)" />
   <xacro:property name="namespace" value="$(arg namespace)" />
+  <xacro:property name="is_public_sim" value="$(arg is_public_sim)" />
   <!-- INCLUDES -->
   <!-- Tools -->
